Commit message: spaces

File: src/viam/sdk/tests/testfiles/gp12.urdf (robot description, URDF)
Before this commit: robot motoman_gp12, 8 links, 7 joints
Joints:
- joint joint_6_t-tool0: type fixed -> None

Commit message: whoops

File: src/viam/sdk/tests/testfiles/gp12.urdf (robot description, URDF)
Before this commit: robot motoman_gp12, 8 links, 7 joints
Joints:
- joint joint_6_t-tool0: type None -> fixed
